File: pcb/beyblock20/beyblock20.kicad_sch (KiCad schematic)
At the start: 43 parts

Commit message: board init
Parts:
- added OL1, OL2: OLED, kbd:OLED_v2, symbol kbd:OLED
- D1: renamed from D?; value (none) -> LL4148; footprint (none) -> Diode_SMD:D_MiniMELF
- J1: renamed from J?; value (none) -> Conn_01x04_Female; footprint (none) -> Connector_PinSocket_2.54mm:PinSocket_1x04_P2.54mm_Vertical
- J2: renamed from J?; value (none) -> Conn_01x04_Male; footprint (none) -> Connector_PinHeader_2.54mm:PinHeader_1x04_P2.54mm_Vertical
- SW1: renamed from SW?; value (none) -> SW_SPST; footprint (none) -> keyswitches:Kailh_socket_MX
- SW10, SW11, SW12, SW13, SW14, SW15, SW16, SW17, SW18, SW19, SW2, SW20, SW3, SW4, SW5, SW6, SW7, SW8, SW9: renamed from SW?; footprint (none) -> keyswitches:Kailh_socket_MX
- U1: renamed from U?; value (none) -> SeeeduinoXIAO; footprint (none) -> Seeeduino XIAO KICAD:Seeeduino XIAO-MOUDLE14P-2.54-21X17.8MM
- gave numbers to parts that had none: 19
Connections:
- net 3v3: now also OL1.3 (VCC), OL2.3 (VCC)
- net gnd: now also J1.3 (Pin_3), J2.3 (Pin_3), OL1.4 (GND), OL2.4 (GND); no longer J1.1 (Pin_1), J2.1 (Pin_1)
- net scl: now also J1.1 (Pin_1), J2.1 (Pin_1), OL1.2 (SCL), OL2.2 (SCL); no longer J1.2 (Pin_2), J2.2 (Pin_2)
- net sda: now also J1.2 (Pin_2), J2.2 (Pin_2), OL1.1 (SDA), OL2.1 (SDA); no longer J1.3 (Pin_3), J2.3 (Pin_3)

Commit message: finish initial pcb
Parts:
- added H1, H2, H3, H4, H5, H6, H7, H8: MountingHole, symbol Mechanical:MountingHole
Connections:
- net 3v3: now also J1.3 (Pin_3), J2.3 (Pin_3); no longer J1.4 (Pin_4), J2.4 (Pin_4)
- net gnd: now also J1.4 (Pin_4), J2.4 (Pin_4); no longer J1.3 (Pin_3), J2.3 (Pin_3)
- net scl: now also J1.2 (Pin_2), J2.2 (Pin_2); no longer J1.1 (Pin_1), J2.1 (Pin_1)
- net sda: now also J1.1 (Pin_1), J2.1 (Pin_1); no longer J1.2 (Pin_2), J2.2 (Pin_2)
Other:
- moved on the sheet: J1, J2

Commit message: add trrs
Parts:
- added U2: (no value), symbol keebio:TRRS
- added U3: TRRS, symbol keebio:TRRS
- H1, H2, H3, H4, H5, H6, H7, H8: footprint (none) -> MountingHole:MountingHole_2.2mm_M2
Connections:
- net 3v3: now also U2.2 (TIP), U3.2 (TIP)
- net gnd: now also U2.1 (SLEEVE), U3.1 (SLEEVE)
- net scl: now also U2.3 (RING1), U3.3 (RING1)
- net sda: now also U2.4 (RING2), U3.4 (RING2)
Changed lines of the file:
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@@
+    )
+  )
+  (global_label "scl" (shape input) (at 133.35 128.27 180) (fields_autoplaced)
+    (effects (font (size 1.27 1.27)) (justify right))
+    (property "Intersheet References" "${INTERSHEET_REFS}" (id 0) (at 128.155 128.1906 0)
+      (effects (font (size 1.27 1.27)) (justify right) hide)
     )
   )
@@
     )
   )
+  (global_label "sda" (shape input) (at 109.22 130.81 180) (fields_autoplaced)
+    (effects (font (size 1.27 1.27)) (justify right))
+    (property "Intersheet References" "${INTERSHEET_REFS}" (id 0) (at 103.4807 130.7306 0)
+      (effects (font (size 1.27 1.27)) (justify right) hide)
+    )
+  )
   (global_label "gnd" (shape input) (at 48.26 175.26 180) (fields_autoplaced)
     (effects (font (size 1.27 1.27)) (justify right))
@@
     )
   )
+  (global_label "sda" (shape input) (at 133.35 130.81 180) (fields_autoplaced)
+    (effects (font (size 1.27 1.27)) (justify right))
+    (property "Intersheet References" "${INTERSHEET_REFS}" (id 0) (at 127.6107 130.7306 0)
+      (effects (font (size 1.27 1.27)) (justify right) hide)
+    )
+  )
+  (global_label "3v3" (shape input) (at 109.22 125.73 180) (fields_autoplaced)
+    (effects (font (size 1.27 1.27)) (justify right))
+    (property "Intersheet References" "${INTERSHEET_REFS}" (id 0) (at 103.4202 125.6506 0)
+      (effects (font (size 1.27 1.27)) (justify right) hide)
+    )
+  )
+  (global_label "scl" (shape input) (at 109.22 128.27 180) (fields_autoplaced)
+    (effects (font (size 1.27 1.27)) (justify right))
+    (property "Intersheet References" "${INTERSHEET_REFS}" (id 0) (at 104.025 128.1906 0)
+      (effects (font (size 1.27 1.27)) (justify right) hide)
+    )
+  )
   (global_label "row4" (shape output) (at 109.22 107.95 180) (fields_autoplaced)
     (effects (font (size 1.27 1.27)) (justify right))
@@
     (effects (font (size 1.27 1.27)) (justify right))
     (property "Intersheet References" "${INTERSHEET_REFS}" (id 0) (at 23.9545 40.5606 0)
+      (effects (font (size 1.27 1.27)) (justify right) hide)
+    )
+  )
+  (global_label "3v3" (shape input) (at 133.35 125.73 180) (fields_autoplaced)
+    (effects (font (size 1.27 1.27)) (justify right))
+    (property "Intersheet References" "${INTERSHEET_REFS}" (id 0) (at 127.5502 125.6506 0)
       (effects (font (size 1.27 1.27)) (justify right) hide)
     )
@@
     )
   )
+  (global_label "gnd" (shape input) (at 133.35 133.35 180) (fields_autoplaced)
+    (effects (font (size 1.27 1.27)) (justify right))
+    (property "Intersheet References" "${INTERSHEET_REFS}" (id 0) (at 127.4898 133.2706 0)
+      (effects (font (size 1.27 1.27)) (justify right) hide)
+    )
+  )
   (global_label "row3" (shape input) (at 72.39 52.07 0) (fields_autoplaced)
     (effects (font (size 1.27 1.27)) (justify left))
@@
     )
   )
+  (global_label "gnd" (shape input) (at 109.22 133.35 180) (fields_autoplaced)
+    (effects (font (size 1.27 1.27)) (justify right))
+    (property "Intersheet References" "${INTERSHEET_REFS}" (id 0) (at 103.3598 133.2706 0)
+      (effects (font (size 1.27 1.27)) (justify right) hide)
+    )
+  )
   (global_label "scl" (shape input) (at 48.26 167.64 180) (fields_autoplaced)
     (effects (font (size 1.27 1.27)) (justify right))
@@
     (pin "2")
   )
+  (symbol (lib_id "keebio:TRRS") (at 118.11 135.89 0) (unit 1)
+    (in_bom yes) (on_board yes) (fields_autoplaced)
+    (property "Reference" "U2" (id 0) (at 123.825 128.5638 0)
+      (effects (font (size 1.524 1.524)) (justify left))
+    )
+    (property "Value" "" (id 1) (at 123.825 131.5572 0)
+      (effects (font (size 1.524 1.524)) (justify left))
+    )
+    (property "Footprint" "" (id 2) (at 121.92 135.89 0)
+      (effects (font (size 1.524 1.524)) hide)
+    )
+    (property "Datasheet" "" (id 3) (at 121.92 135.89 0)
+      (effects (font (size 1.524 1.524)) hide)
+    )
+    (pin "1")
+    (pin "2")
+    (pin "3")
+    (pin "4")
+  )
   (symbol (lib_id "Diode:LL4148") (at 115.57 63.5 90) (unit 1)
     (in_bom yes) (on_board yes) (fields_autoplaced)
@@
       (effects (font (size 1.27 1.27)) (justify left))
     )
-    (property "Footprint" "" (id 2) (at 115.57 114.3 0)
+    (property "Footprint" "MountingHole:MountingHole_2.2mm_M2" (id 2) (at 115.57 114.3 0)
       (effects (font (size 1.27 1.27)) hide)
     )
@@
     (pin "2")
   )
+  (symbol (lib_id "keebio:TRRS") (at 142.24 135.89 0) (unit 1)
+    (in_bom yes) (on_board yes) (fields_autoplaced)
+    (property "Reference" "U3" (id 0) (at 147.955 128.5638 0)
+      (effects (font (size 1.524 1.524)) (justify left))
+    )
+    (property "Value" "TRRS" (id 1) (at 147.955 131.5572 0)
+      (effects (font (size 1.524 1.524)) (justify left))
+    )
+    (property "Footprint" "" (id 2) (at 146.05 135.89 0)
+      (effects (font (size 1.524 1.524)) hide)
+    )
+    (property "Datasheet" "" (id 3) (at 146.05 135.89 0)
+      (effects (font (size 1.524 1.524)) hide)
+    )
+    (pin "1")
+    (pin "2")
+    (pin "3")
+    (pin "4")
+  )
   (symbol (lib_id "Switch:SW_SPST") (at 133.35 80.01 0) (unit 1)
     (in_bom yes) (on_board yes) (fields_autoplaced)
@@
       (effects (font (size 1.27 1.27)) (justify left))
     )
-    (property "Footprint" "" (id 2) (at 60.96 182.88 0)
+    (property "Footprint" "MountingHole:MountingHole_2.2mm_M2" (id 2) (at 60.96 182.88 0)
       (effects (font (size 1.27 1.27)) hide)
     )
@@
       (effects (font (size 1.27 1.27)) (justify left))
     )
-    (property "Footprint" "" (id 2) (at 121.92 114.3 0)
+    (property "Footprint" "MountingHole:MountingHole_2.2mm_M2" (id 2) (at 121.92 114.3 0)
       (effects (font (size 1.27 1.27)) hide)
     )
@@
       (effects (font (size 1.27 1.27)) (justify left))
     )
-    (property "Footprint" "" (id 2) (at 134.62 114.3 0)
+    (property "Footprint" "MountingHole:MountingHole_2.2mm_M2" (id 2) (at 134.62 114.3 0)
       (effects (font (size 1.27 1.27)) hide)
     )
@@
       (effects (font (size 1.27 1.27)) (justify left))
     )
-    (property "Footprint" "" (id 2) (at 67.31 182.88 0)
+    (property "Footprint" "MountingHole:MountingHole_2.2mm_M2" (id 2) (at 67.31 182.88 0)
       (effects (font (size 1.27 1.27)) hide)
     )
@@
       (effects (font (size 1.27 1.27)) (justify left))
     )
-    (property "Footprint" "" (id 2) (at 54.61 182.88 0)
+    (property "Footprint" "MountingHole:MountingHole_2.2mm_M2" (id 2) (at 54.61 182.88 0)
       (effects (font (size 1.27 1.27)) hide)
     )
@@
       (effects (font (size 1.27 1.27)) (justify left))
     )
-    (property "Footprint" "" (id 2) (at 128.27 114.3 0)
+    (property "Footprint" "MountingHole:MountingHole_2.2mm_M2" (id 2) (at 128.27 114.3 0)
       (effects (font (size 1.27 1.27)) hide)
     )
@@
       (effects (font (size 1.27 1.27)) (justify left))
     )
-    (property "Footprint" "" (id 2) (at 73.66 182.88 0)
+    (property "Footprint" "MountingHole:MountingHole_2.2mm_M2" (id 2) (at 73.66 182.88 0)
       (effects (font (size 1.27 1.27)) hide)
     )
@@
       (reference "U1") (unit 1) (value "SeeeduinoXIAO") (footprint "Seeeduino XIAO KICAD:Seeeduino XIAO-MOUDLE14P-2.54-21X17.8MM")
     )
-  )
+    (path "/1440444c-7b3c-4048-bee5-f38a07cb6ccb"
+      (reference "U2") (unit 1) (value "TRRS") (footprint "Keebio-Parts:TRRS-PJ-320A")
+    )
+    (path "/5c2f63e8-3854-47c2-b529-57fcc99ef42d"
+      (reference "U3") (unit 1) (value "TRRS") (footprint "Keebio-Parts:TRRS-PJ-320A")
+    )
+  )

Commit message: update beyblock20 and knoblin3
Parts:
- added C1, C2: C, Capacitor_SMD:C_Elec_6.3x5.8, symbol Device:C
- added R1, R2: R, symbol Device:R
- U2: value (none) -> TRRS; footprint (none) -> Keebio-Parts:TRRS-PJ-320A
- U3: footprint (none) -> Keebio-Parts:TRRS-PJ-320A
Connections:
- net 3v3: now also C1.1, C2.1, R1.1, R2.1
- net gnd: now also C1.2, C2.2
- net scl: now also R2.2
- net sda: now also R1.2
Other:
- note added: "Decoupling Capacitor Used to mitigate against brownout"
- note added: "I2C pullup resistors (To be used if screen is not used)"
Changed lines of the file:
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@@
+    (stroke (width 0) (type default) (color 0 0 0 0))
+  )
+  (wire (pts (xy 123.19 163.83) (xy 125.73 163.83))
     (stroke (width 0) (type default) (color 0 0 0 0))
   )
@@
     (stroke (width 0) (type default) (color 0 0 0 0))
   )
+  (wire (pts (xy 123.19 168.91) (xy 125.73 168.91))
+    (stroke (width 0) (type default) (color 0 0 0 0))
+  )
   (wire (pts (xy 140.97 46.99) (xy 153.67 46.99))
     (stroke (width 0) (type default) (color 0 0 0 0))
@@
     (stroke (width 0) (type default) (color 0 0 0 0))
   )
+  (wire (pts (xy 133.35 168.91) (xy 135.89 168.91))
+    (stroke (width 0) (type default) (color 0 0 0 0))
+  )
   (wire (pts (xy 125.73 59.69) (xy 125.73 80.01))
     (stroke (width 0) (type default) (color 0 0 0 0))
@@
     (stroke (width 0) (type default) (color 0 0 0 0))
   )
+  (wire (pts (xy 133.35 163.83) (xy 135.89 163.83))
+    (stroke (width 0) (type default) (color 0 0 0 0))
+  )
   (wire (pts (xy 109.22 87.63) (xy 115.57 87.63))
     (stroke (width 0) (type default) (color 0 0 0 0))
@@
     (stroke (width 0) (type default) (color 0 0 0 0))
   )
+  (text "I2C pullup resistors\n(To be used if screen is not used)"
+    (at 120.65 157.48 0)
+    (effects (font (size 1.27 1.27)) (justify left bottom))
+  )
+  (text "Decoupling Capacitor\nUsed to mitigate against brownout"
+    (at 54.61 99.06 0)
+    (effects (font (size 1.27 1.27)) (justify left bottom))
+  )
   (global_label "gnd" (shape input) (at 48.26 157.48 180) (fields_autoplaced)
     (effects (font (size 1.27 1.27)) (justify right))
@@
     )
   )
+  (global_label "3v3" (shape input) (at 123.19 168.91 180) (fields_autoplaced)
+    (effects (font (size 1.27 1.27)) (justify right))
+    (property "Intersheet References" "${INTERSHEET_REFS}" (id 0) (at 117.3902 168.8306 0)
+      (effects (font (size 1.27 1.27)) (justify right) hide)
+    )
+  )
   (global_label "col4" (shape output) (at 30.48 44.45 180) (fields_autoplaced)
     (effects (font (size 1.27 1.27)) (justify right))
@@
     )
   )
+  (global_label "sda" (shape input) (at 135.89 163.83 0) (fields_autoplaced)
+    (effects (font (size 1.27 1.27)) (justify left))
+    (property "Intersheet References" "${INTERSHEET_REFS}" (id 0) (at 141.6293 163.7506 0)
+      (effects (font (size 1.27 1.27)) (justify left) hide)
+    )
+  )
+  (global_label "scl" (shape input) (at 135.89 168.91 0) (fields_autoplaced)
+    (effects (font (size 1.27 1.27)) (justify left))
+    (property "Intersheet References" "${INTERSHEET_REFS}" (id 0) (at 141.085 168.8306 0)
+      (effects (font (size 1.27 1.27)) (justify left) hide)
+    )
+  )
   (global_label "scl" (shape input) (at 133.35 128.27 180) (fields_autoplaced)
     (effects (font (size 1.27 1.27)) (justify right))
@@
     )
   )
+  (global_label "3v3" (shape input) (at 123.19 163.83 180) (fields_autoplaced)
+    (effects (font (size 1.27 1.27)) (justify right))
+    (property "Intersheet References" "${INTERSHEET_REFS}" (id 0) (at 117.3902 163.7506 0)
+      (effects (font (size 1.27 1.27)) (justify right) hide)
+    )
+  )
   (global_label "sda" (shape output) (at 30.48 48.26 180) (fields_autoplaced)
     (effects (font (size 1.27 1.27)) (justify right))
@@
     )
   )
+  (global_label "gnd" (shape input) (at 48.26 113.03 180) (fields_autoplaced)
+    (effects (font (size 1.27 1.27)) (justify right))
+    (property "Intersheet References" "${INTERSHEET_REFS}" (id 0) (at 42.3998 112.9506 0)
+      (effects (font (size 1.27 1.27)) (justify right) hide)
+    )
+  )
   (global_label "3v3" (shape input) (at 48.26 171.45 180) (fields_autoplaced)
     (effects (font (size 1.27 1.27)) (justify right))
@@
     )
   )
+  (global_label "gnd" (shape input) (at 48.26 101.6 180) (fields_autoplaced)
+    (effects (font (size 1.27 1.27)) (justify right))
+    (property "Intersheet References" "${INTERSHEET_REFS}" (id 0) (at 42.3998 101.5206 0)
+      (effects (font (size 1.27 1.27)) (justify right) hide)
+    )
+  )
   (global_label "scl" (shape input) (at 109.22 128.27 180) (fields_autoplaced)
     (effects (font (size 1.27 1.27)) (justify right))
@@
     )
   )
+  (global_label "3v3" (shape input) (at 48.26 105.41 180) (fields_autoplaced)
+    (effects (font (size 1.27 1.27)) (justify right))
+    (property "Intersheet References" "${INTERSHEET_REFS}" (id 0) (at 42.4602 105.3306 0)
+      (effects (font (size 1.27 1.27)) (justify right) hide)
+    )
+  )
   (global_label "row3" (shape output) (at 109.22 87.63 180) (fields_autoplaced)
     (effects (font (size 1.27 1.27)) (justify right))
@@
     (property "Intersheet References" "${INTERSHEET_REFS}" (id 0) (at 163.7506 25.2245 90)
       (effects (font (size 1.27 1.27)) (justify left) hide)
+    )
+  )
+  (global_label "3v3" (shape input) (at 48.26 93.98 180) (fields_autoplaced)
+    (effects (font (size 1.27 1.27)) (justify right))
+    (property "Intersheet References" "${INTERSHEET_REFS}" (id 0) (at 42.4602 93.9006 0)
+      (effects (font (size 1.27 1.27)) (justify right) hide)
     )
   )
@@
       (effects (font (size 1.524 1.524)) (justify left))
     )
-    (property "Value" "" (id 1) (at 123.825 131.5572 0)
+    (property "Value" "TRRS" (id 1) (at 123.825 131.5572 0)
       (effects (font (size 1.524 1.524)) (justify left))
     )
-    (property "Footprint" "" (id 2) (at 121.92 135.89 0)
+    (property "Footprint" "Keebio-Parts:TRRS-PJ-320A" (id 2) (at 121.92 135.89 0)
       (effects (font (size 1.524 1.524)) hide)
     )
@@
     (pin "4")
   )
+  (symbol (lib_id "Device:R") (at 129.54 168.91 90) (unit 1)
+    (in_bom yes) (on_board yes) (fields_autoplaced)
+    (property "Reference" "R2" (id 0) (at 129.54 164.1942 90))
+    (property "Value" "R" (id 1) (at 129.54 166.7311 90))
+    (property "Footprint" "" (id 2) (at 129.54 170.688 90)
+      (effects (font (size 1.27 1.27)) hide)
+    )
+    (property "Datasheet" "~" (id 3) (at 129.54 168.91 0)
+      (effects (font (size 1.27 1.27)) hide)
+    )
+    (pin "1")
+    (pin "2")
+  )
   (symbol (lib_id "Switch:SW_SPST") (at 133.35 100.33 0) (unit 1)
     (in_bom yes) (on_board yes) (fields_autoplaced)
@@
     (pin "2")
   )
+  (symbol (lib_id "Device:R") (at 129.54 163.83 90) (unit 1)
+    (in_bom yes) (on_board yes) (fields_autoplaced)
+    (property "Reference" "R1" (id 0) (at 129.54 159.1142 90))
+    (property "Value" "R" (id 1) (at 129.54 161.6511 90))
+    (property "Footprint" "" (id 2) (at 129.54 165.608 90)
+      (effects (font (size 1.27 1.27)) hide)
+    )
+    (property "Datasheet" "~" (id 3) (at 129.54 163.83 0)
+      (effects (font (size 1.27 1.27)) hide)
+    )
+    (pin "1")
+    (pin "2")
+  )
   (symbol (lib_id "Diode:LL4148") (at 166.37 104.14 90) (unit 1)
     (in_bom yes) (on_board yes) (fields_autoplaced)
@@
       (effects (font (size 1.524 1.524)) (justify left))
     )
-    (property "Footprint" "" (id 2) (at 146.05 135.89 0)
+    (property "Footprint" "Keebio-Parts:TRRS-PJ-320A" (id 2) (at 146.05 135.89 0)
       (effects (font (size 1.524 1.524)) hide)
     )
@@
     (pin "3")
     (pin "4")
+  )
+  (symbol (lib_id "Device:C") (at 48.26 109.22 0) (unit 1)
+    (in_bom yes) (on_board yes) (fields_autoplaced)
+    (property "Reference" "C2" (id 0) (at 51.181 108.3853 0)
+      (effects (font (size 1.27 1.27)) (justify left))
+    )
+    (property "Value" "C" (id 1) (at 51.181 110.9222 0)
+      (effects (font (size 1.27 1.27)) (justify left))
+    )
+    (property "Footprint" "Capacitor_SMD:C_Elec_6.3x5.8" (id 2) (at 49.2252 113.03 0)
+      (effects (font (size 1.27 1.27)) hide)
+    )
+    (property "Datasheet" "~" (id 3) (at 48.26 109.22 0)
+      (effects (font (size 1.27 1.27)) hide)
+    )
+    (pin "1")
+    (pin "2")
   )
   (symbol (lib_id "Switch:SW_SPST") (at 133.35 80.01 0) (unit 1)
@@
     (pin "2")
   )
+  (symbol (lib_id "Device:C") (at 48.26 97.79 0) (unit 1)
+    (in_bom yes) (on_board yes) (fields_autoplaced)
+    (property "Reference" "C1" (id 0) (at 51.181 96.9553 0)
+      (effects (font (size 1.27 1.27)) (justify left))
+    )
+    (property "Value" "C" (id 1) (at 51.181 99.4922 0)
+      (effects (font (size 1.27 1.27)) (justify left))
+    )
+    (property "Footprint" "Capacitor_SMD:C_Elec_6.3x5.8" (id 2) (at 49.2252 101.6 0)
+      (effects (font (size 1.27 1.27)) hide)
+    )
+    (property "Datasheet" "~" (id 3) (at 48.26 97.79 0)
+      (effects (font (size 1.27 1.27)) hide)
+    )
+    (pin "1")
+    (pin "2")
+  )
   (symbol (lib_id "Switch:SW_SPST") (at 158.75 59.69 0) (unit 1)
     (in_bom yes) (on_board yes) (fields_autoplaced)
@@
   )
   (symbol_instances
+    (path "/be38b6b4-07fe-46cb-9636-991ca80eb1da"
+      (reference "C1") (unit 1) (value "C") (footprint "Capacitor_SMD:C_Elec_6.3x5.8")
+    )
+    (path "/6159ee8f-0142-40f0-9b87-f7bec106aabd"
+      (reference "C2") (unit 1) (value "C") (footprint "Capacitor_SMD:C_Elec_6.3x5.8")
+    )
     (path "/9d18ea08-acf0-40b3-a16d-62401a5ff325"
       (reference "D1") (unit 1) (value "LL4148") (footprint "Diode_SMD:D_MiniMELF")
@@
       (reference "OL2") (unit 1) (value "OLED") (footprint "kbd:OLED_v2")
     )
+    (path "/5926988a-09d8-483f-9cc9-6831ce2c56ad"
+      (reference "R1") (unit 1) (value "R") (footprint "Resistor_SMD:R_1206_3216Metric_Pad1.30x1.75mm_HandSolder")
+    )
+    (path "/44475545-1d14-4435-9d00-5dd22a27985c"
+      (reference "R2") (unit 1) (value "R") (footprint "Resistor_SMD:R_1206_3216Metric_Pad1.30x1.75mm_HandSolder")
+    )
     (path "/96d03886-47df-4a69-935b-56c4327baad1"
