File: pcb/beyblock20/beyblock20.kicad_sch (KiCad schematic)
At the start: 59 parts, among them J1 Conn_01x04_Female, J2 Conn_01x04_Male, SW1 SW_SPST, SW10 SW_SPST, SW11 SW_SPST, SW12 SW_SPST, SW13 SW_SPST, SW14 SW_SPST, SW15 SW_SPST, SW16 SW_SPST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

Commit message: add mongus48. make beyblock updates
Parts:
- removed C1, C2: C, Capacitor_SMD:C_Elec_6.3x5.8, symbol Device:C
- added C1, C2: (no value), symbol Device:C_Polarized_US
- R1, R2: footprint (none) -> Resistor_SMD:R_1206_3216Metric_Pad1.30x1.75mm_HandSolder
Connections:
- net 3v3 renamed +3V3
- net +3V3: now also C1.1, C2.1
- net gnd renamed GND
- net GND: now also C1.2, C2.2
Changed lines of the file:
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@@
     )
   )
-  (global_label "gnd" (shape input) (at 48.26 113.03 180) (fields_autoplaced)
-    (effects (font (size 1.27 1.27)) (justify right))
-    (property "Intersheet References" "${INTERSHEET_REFS}" (id 0) (at 42.3998 112.9506 0)
+  (global_label "gnd" (shape input) (at 48.26 119.38 180) (fields_autoplaced)
+    (effects (font (size 1.27 1.27)) (justify right))
+    (property "Intersheet References" "${INTERSHEET_REFS}" (id 0) (at 42.3998 119.3006 0)
       (effects (font (size 1.27 1.27)) (justify right) hide)
     )
@@
     )
   )
-  (global_label "3v3" (shape input) (at 48.26 105.41 180) (fields_autoplaced)
-    (effects (font (size 1.27 1.27)) (justify right))
-    (property "Intersheet References" "${INTERSHEET_REFS}" (id 0) (at 42.4602 105.3306 0)
+  (global_label "3v3" (shape input) (at 48.26 111.76 180) (fields_autoplaced)
+    (effects (font (size 1.27 1.27)) (justify right))
+    (property "Intersheet References" "${INTERSHEET_REFS}" (id 0) (at 42.4602 111.6806 0)
       (effects (font (size 1.27 1.27)) (justify right) hide)
     )
@@
     (pin "2")
   )
+  (symbol (lib_id "power:+3.3V") (at 48.26 93.98 0) (unit 1)
+    (in_bom yes) (on_board yes) (fields_autoplaced)
+    (property "Reference" "#PWR0101" (id 0) (at 48.26 97.79 0)
+      (effects (font (size 1.27 1.27)) hide)
+    )
+    (property "Value" "" (id 1) (at 48.26 90.4042 0))
+    (property "Footprint" "" (id 2) (at 48.26 93.98 0)
+      (effects (font (size 1.27 1.27)) hide)
+    )
+    (property "Datasheet" "" (id 3) (at 48.26 93.98 0)
+      (effects (font (size 1.27 1.27)) hide)
+    )
+    (pin "1")
+  )
   (symbol (lib_id "Diode:LL4148") (at 153.67 83.82 90) (unit 1)
     (in_bom yes) (on_board yes) (fields_autoplaced)
@@
     (property "Reference" "R2" (id 0) (at 129.54 164.1942 90))
     (property "Value" "R" (id 1) (at 129.54 166.7311 90))
-    (property "Footprint" "" (id 2) (at 129.54 170.688 90)
+    (property "Footprint" "Resistor_SMD:R_1206_3216Metric_Pad1.30x1.75mm_HandSolder" (id 2) (at 129.54 170.688 90)
       (effects (font (size 1.27 1.27)) hide)
     )
@@
     (property "Reference" "R1" (id 0) (at 129.54 159.1142 90))
     (property "Value" "R" (id 1) (at 129.54 161.6511 90))
-    (property "Footprint" "" (id 2) (at 129.54 165.608 90)
+    (property "Footprint" "Resistor_SMD:R_1206_3216Metric_Pad1.30x1.75mm_HandSolder" (id 2) (at 129.54 165.608 90)
       (effects (font (size 1.27 1.27)) hide)
     )
@@
     (pin "3")
     (pin "4")
-  )
-  (symbol (lib_id "Device:C") (at 48.26 109.22 0) (unit 1)
-    (in_bom yes) (on_board yes) (fields_autoplaced)
-    (property "Reference" "C2" (id 0) (at 51.181 108.3853 0)
-      (effects (font (size 1.27 1.27)) (justify left))
-    )
-    (property "Value" "C" (id 1) (at 51.181 110.9222 0)
-      (effects (font (size 1.27 1.27)) (justify left))
-    )
-    (property "Footprint" "Capacitor_SMD:C_Elec_6.3x5.8" (id 2) (at 49.2252 113.03 0)
-      (effects (font (size 1.27 1.27)) hide)
-    )
-    (property "Datasheet" "~" (id 3) (at 48.26 109.22 0)
-      (effects (font (size 1.27 1.27)) hide)
-    )
-    (pin "1")
-    (pin "2")
   )
   (symbol (lib_id "Switch:SW_SPST") (at 133.35 80.01 0) (unit 1)
@@
     (pin "2")
   )
+  (symbol (lib_id "power:GND") (at 48.26 119.38 0) (unit 1)
+    (in_bom yes) (on_board yes) (fields_autoplaced)
+    (property "Reference" "#PWR0104" (id 0) (at 48.26 125.73 0)
+      (effects (font (size 1.27 1.27)) hide)
+    )
+    (property "Value" "" (id 1) (at 48.26 123.8234 0))
+    (property "Footprint" "" (id 2) (at 48.26 119.38 0)
+      (effects (font (size 1.27 1.27)) hide)
+    )
+    (property "Datasheet" "" (id 3) (at 48.26 119.38 0)
+      (effects (font (size 1.27 1.27)) hide)
+    )
+    (pin "1")
+  )
   (symbol (lib_id "Switch:SW_SPST") (at 146.05 39.37 0) (unit 1)
     (in_bom yes) (on_board yes) (fields_autoplaced)
@@
     (pin "1")
     (pin "2")
+  )
+  (symbol (lib_id "power:GND") (at 48.26 101.6 0) (unit 1)
+    (in_bom yes) (on_board yes)
+    (property "Reference" "#PWR0102" (id 0) (at 48.26 107.95 0)
+      (effects (font (size 1.27 1.27)) hide)
+    )
+    (property "Value" "" (id 1) (at 48.26 112.3934 0))
+    (property "Footprint" "" (id 2) (at 48.26 101.6 0)
+      (effects (font (size 1.27 1.27)) hide)
+    )
+    (property "Datasheet" "" (id 3) (at 48.26 101.6 0)
+      (effects (font (size 1.27 1.27)) hide)
+    )
+    (pin "1")
   )
   (symbol (lib_id "Mechanical:MountingHole") (at 60.96 182.88 0) (unit 1)
@@
     )
   )
+  (symbol (lib_id "power:+3.3V") (at 48.26 111.76 0) (unit 1)
+    (in_bom yes) (on_board yes) (fields_autoplaced)
+    (property "Reference" "#PWR0103" (id 0) (at 48.26 115.57 0)
+      (effects (font (size 1.27 1.27)) hide)
+    )
+    (property "Value" "" (id 1) (at 48.26 108.1842 0))
+    (property "Footprint" "" (id 2) (at 48.26 111.76 0)
+      (effects (font (size 1.27 1.27)) hide)
+    )
+    (property "Datasheet" "" (id 3) (at 48.26 111.76 0)
+      (effects (font (size 1.27 1.27)) hide)
+    )
+    (pin "1")
+  )
   (symbol (lib_id "Diode:LL4148") (at 128.27 43.18 90) (unit 1)
     (in_bom yes) (on_board yes) (fields_autoplaced)
@@
     (pin "2")
   )
+  (symbol (lib_id "Device:C_Polarized_US") (at 48.26 115.57 0) (unit 1)
+    (in_bom yes) (on_board yes) (fields_autoplaced)
+    (property "Reference" "C2" (id 0) (at 51.181 114.1003 0)
+      (effects (font (size 1.27 1.27)) (justify left))
+    )
+    (property "Value" "" (id 1) (at 51.181 116.6372 0)
+      (effects (font (size 1.27 1.27)) (justify left))
+    )
+    (property "Footprint" "" (id 2) (at 48.26 115.57 0)
+      (effects (font (size 1.27 1.27)) hide)
+    )
+    (property "Datasheet" "~" (id 3) (at 48.26 115.57 0)
+      (effects (font (size 1.27 1.27)) hide)
+    )
+    (pin "1")
+    (pin "2")
+  )
   (symbol (lib_id "Switch:SW_SPST") (at 146.05 59.69 0) (unit 1)
     (in_bom yes) (on_board yes) (fields_autoplaced)
@@
     (pin "2")
   )
-  (symbol (lib_id "Device:C") (at 48.26 97.79 0) (unit 1)
-    (in_bom yes) (on_board yes) (fields_autoplaced)
-    (property "Reference" "C1" (id 0) (at 51.181 96.9553 0)
-      (effects (font (size 1.27 1.27)) (justify left))
-    )
-    (property "Value" "C" (id 1) (at 51.181 99.4922 0)
-      (effects (font (size 1.27 1.27)) (justify left))
-    )
-    (property "Footprint" "Capacitor_SMD:C_Elec_6.3x5.8" (id 2) (at 49.2252 101.6 0)
-      (effects (font (size 1.27 1.27)) hide)
-    )
-    (property "Datasheet" "~" (id 3) (at 48.26 97.79 0)
-      (effects (font (size 1.27 1.27)) hide)
-    )
-    (pin "1")
-    (pin "2")
-  )
   (symbol (lib_id "Switch:SW_SPST") (at 158.75 59.69 0) (unit 1)
     (in_bom yes) (on_board yes) (fields_autoplaced)
@@
     (pin "2")
   )
+  (symbol (lib_id "Device:C_Polarized_US") (at 48.26 97.79 0) (unit 1)
+    (in_bom yes) (on_board yes) (fields_autoplaced)
+    (property "Reference" "C1" (id 0) (at 51.181 96.3203 0)
+      (effects (font (size 1.27 1.27)) (justify left))
+    )
+    (property "Value" "" (id 1) (at 51.181 98.8572 0)
+      (effects (font (size 1.27 1.27)) (justify left))
+    )
+    (property "Footprint" "" (id 2) (at 48.26 97.79 0)
+      (effects (font (size 1.27 1.27)) hide)
+    )
+    (property "Datasheet" "~" (id 3) (at 48.26 97.79 0)
+      (effects (font (size 1.27 1.27)) hide)
+    )
+    (pin "1")
+    (pin "2")
+  )
   (symbol (lib_id "Diode:LL4148") (at 166.37 63.5 90) (unit 1)
     (in_bom yes) (on_board yes) (fields_autoplaced)
@@
   )
   (symbol_instances
-    (path "/be38b6b4-07fe-46cb-9636-991ca80eb1da"
-      (reference "C1") (unit 1) (value "C") (footprint "Capacitor_SMD:C_Elec_6.3x5.8")
-    )
-    (path "/6159ee8f-0142-40f0-9b87-f7bec106aabd"
-      (reference "C2") (unit 1) (value "C") (footprint "Capacitor_SMD:C_Elec_6.3x5.8")
+    (path "/2f7e0016-8ef9-44a8-b4ce-24c46355aa1e"
+      (reference "#PWR0101") (unit 1) (value "+3.3V") (footprint "")
+    )
+    (path "/76a16b35-d931-4996-8938-9da762e9492c"
+      (reference "#PWR0102") (unit 1) (value "GND") (footprint "")
+    )
+    (path "/92367d55-e866-4d69-84fa-bb361751d6c6"
+      (reference "#PWR0103") (unit 1) (value "+3.3V") (footprint "")
+    )
+    (path "/6f8abb20-d786-4404-9a62-dea63c774b5f"
+      (reference "#PWR0104") (unit 1) (value "GND") (footprint "")
+    )
+    (path "/edb5bb03-4415-4623-9d67-27f3fb66bc32"
+      (reference "C1") (unit 1) (value "C_Polarized_US") (footprint "Capacitor_SMD:CP_Elec_6.3x7.7")
+    )
+    (path "/aa07ccab-65da-4072-99a9-9fbd288c7e56"
+      (reference "C2") (unit 1) (value "C_Polarized_US") (footprint "Capacitor_SMD:CP_Elec_6.3x7.7")
     )
     (path "/9d18ea08-acf0-40b3-a16d-62401a5ff325"
