File: pcb/mongus48/mongus48.kicad_sch (KiCad schematic)
At the start: 120 parts, among them J3 Conn_01x04_Male, J4 Conn_01x04_Female, SW1 RotaryEncoder_Switch, SW10 SW_SPST, SW11 SW_SPST, SW12 SW_SPST, SW13 SW_SPST, SW14 SW_SPST, SW15 SW_SPST, SW16 SW_SPST, SW17 SW_SPST, SW18 SW_SPST, SW19 SW_SPST, SW2 SW_SPST, SW20 SW_SPST, SW21 SW_SPST, SW22 SW_SPST, SW23 SW_SPST, SW24 SW_SPST, SW25 SW_SPST, SW26 SW_SPST, SW27 SW_SPST, SW28 SW_SPST, SW29 SW_SPST, SW3 SW_SPST, SW30 SW_SPST, SW31 SW_SPST, SW32 SW_SPST, SW33 SW_SPST, SW34 SW_SPST, SW35 SW_SPST, SW36 SW_SPST, SW37 SW_SPST, SW38 SW_SPST, SW39 SW_SPST, SW4 SW_SPST, SW40 SW_SPST, SW41 SW_SPST, SW42 SW_SPST, SW43 SW_SPST, SW44 SW_SPST, SW45 SW_SPST, SW46 SW_SPST, SW47 SW_SPST, SW48 SW_SPST, SW49 SW_SPST, SW5 SW_SPST, SW50 SW_SPST, SW51 SW_SPST, SW52 SW_SPST, SW6 SW_SPST, SW7 SW_SPST, SW8 SW_SPST, SW9 SW_SPST, U1 SeeeduinoXIAO, U2 74HC595, U3 74HC595

Commit message: add mongus48. make beyblock updates
Parts:
- removed OL2: OLED, symbol kbd:OLED
- added C1: C_Polarized_US, Capacitor_SMD:CP_Elec_6.3x7.7, symbol Device:C_Polarized_US
- added H11, H12: MountingHole, MountingHole:MountingHole_2.2mm_M2_DIN965, symbol Mechanical:MountingHole
- added R1, R2: R, Resistor_SMD:R_1206_3216Metric_Pad1.30x1.75mm_HandSolder, symbol Device:R
- H1, H10, H2, H3, H4, H5, H6, H7, H8, H9: footprint (none) -> MountingHole:MountingHole_2.2mm_M2_DIN965
- J1: renamed from J3; footprint (none) -> Connector_PinHeader_2.54mm:PinHeader_1x04_P2.54mm_Vertical
- J2: renamed from J4; footprint (none) -> Connector_PinHeader_2.54mm:PinHeader_1x04_P2.54mm_Vertical
- OL1: footprint (none) -> kbd:OLED_v2
- RSW1: renamed from SW1; footprint (none) -> Rotary_Encoder:RotaryEncoder_Alps_EC11E-Switch_Vertical_H20mm
- SW1: renamed from SW2; footprint (none) -> keyswitches:Kailh_socket_MX
- SW10: renamed from SW11; footprint (none) -> keyswitches:Kailh_socket_MX
- SW11: renamed from SW12; footprint (none) -> keyswitches:Kailh_socket_MX
- SW12: renamed from SW13; footprint (none) -> keyswitches:Kailh_socket_MX
- SW13: renamed from SW14; footprint (none) -> keyswitches:Kailh_socket_MX
- SW14: renamed from SW15; footprint (none) -> keyswitches:Kailh_socket_MX
- SW15: renamed from SW16; footprint (none) -> keyswitches:Kailh_socket_MX
- SW16: renamed from SW17; footprint (none) -> keyswitches:Kailh_socket_MX
- SW17: renamed from SW18; footprint (none) -> keyswitches:Kailh_socket_MX
- SW18: renamed from SW19; footprint (none) -> keyswitches:Kailh_socket_MX
- SW19: renamed from SW20; footprint (none) -> keyswitches:Kailh_socket_MX
- SW2: renamed from SW3; footprint (none) -> keyswitches:Kailh_socket_MX
- SW20: renamed from SW21; footprint (none) -> keyswitches:Kailh_socket_MX
- SW21: renamed from SW22; footprint (none) -> keyswitches:Kailh_socket_MX
- SW22: renamed from SW23; footprint (none) -> keyswitches:Kailh_socket_MX
- SW23: renamed from SW24; footprint (none) -> keyswitches:Kailh_socket_MX
- SW24: renamed from SW25; footprint (none) -> keyswitches:Kailh_socket_MX
- SW25: renamed from SW26; footprint (none) -> keyswitches:Kailh_socket_MX
- SW26: renamed from SW27; footprint (none) -> keyswitches:Kailh_socket_MX
- SW27: renamed from SW28; footprint (none) -> keyswitches:Kailh_socket_MX
- SW28: renamed from SW29; footprint (none) -> keyswitches:Kailh_socket_MX
- SW29: renamed from SW30; footprint (none) -> keyswitches:Kailh_socket_MX
- SW3: renamed from SW4; footprint (none) -> keyswitches:Kailh_socket_MX
- SW30: renamed from SW31; footprint (none) -> keyswitches:Kailh_socket_MX
- SW31: renamed from SW32; footprint (none) -> keyswitches:Kailh_socket_MX
- SW32: renamed from SW33; footprint (none) -> keyswitches:Kailh_socket_MX
- SW33: renamed from SW34; footprint (none) -> keyswitches:Kailh_socket_MX
- SW34: renamed from SW35; footprint (none) -> keyswitches:Kailh_socket_MX
- SW35: renamed from SW36; footprint (none) -> keyswitches:Kailh_socket_MX
- SW36: renamed from SW37; footprint (none) -> keyswitches:Kailh_socket_MX
- SW37: renamed from SW41; footprint (none) -> keyswitches:Kailh_socket_MX
- SW38: renamed from SW42; footprint (none) -> keyswitches:Kailh_socket_MX
- SW39: renamed from SW43; footprint (none) -> keyswitches:Kailh_socket_MX
- SW4: renamed from SW5; footprint (none) -> keyswitches:Kailh_socket_MX
- SW40: renamed from SW44; footprint (none) -> keyswitches:Kailh_socket_MX
- SW41: renamed from SW45; footprint (none) -> keyswitches:Kailh_socket_MX
- SW42: renamed from SW39; footprint (none) -> keyswitches:Kailh_socket_MX
- SW43: renamed from SW47; footprint (none) -> keyswitches:Kailh_socket_MX
- SW44: renamed from SW48; footprint (none) -> keyswitches:Kailh_socket_MX
- SW45: renamed from SW49; footprint (none) -> keyswitches:Kailh_socket_MX
- SW46: renamed from SW50; footprint (none) -> keyswitches:Kailh_socket_MX
- SW47: renamed from SW51; footprint (none) -> keyswitches:Kailh_socket_MX
- SW48: renamed from SW52; footprint (none) -> keyswitches:Kailh_socket_MX
- SW49: renamed from SW38; footprint (none) -> keyswitches:Kailh_socket_MX
- SW5: renamed from SW6; footprint (none) -> keyswitches:Kailh_socket_MX
- SW50: renamed from SW40; footprint (none) -> keyswitches:Kailh_socket_MX
- SW51: renamed from SW46; footprint (none) -> keyswitches:Kailh_socket_MX
- SW6: renamed from SW7; footprint (none) -> keyswitches:Kailh_socket_MX
- SW7: renamed from SW8; footprint (none) -> keyswitches:Kailh_socket_MX
- SW8: renamed from SW9; footprint (none) -> keyswitches:Kailh_socket_MX
- SW9: renamed from SW10; footprint (none) -> keyswitches:Kailh_socket_MX
- U1: footprint (none) -> Seeeduino XIAO KICAD:Seeeduino XIAO-MOUDLE14P-2.54-21X17.8MM
- U2: renamed from U3; footprint (none) -> Package_SO:SOP-16_3.9x9.9mm_P1.27mm
- U3: renamed from U2; footprint (none) -> Package_SO:SOP-16_3.9x9.9mm_P1.27mm
- U4, U5: value (none) -> TRRS; footprint (none) -> Keebio-Parts:TRRS-PJ-320A
- renumbered D14 to D13, D15 to D14, D16 to D15, D17 to D16, D18 to D17, D19 to D18, D20 to D19, D21 to D20, D22 to D21, D23 to D22, D24 to D23, D25 to D24, D26 to D25, D27 to D26, D28 to D27, D29 to D28, D30 to D29, D31 to D30, D32 to D31, D33 to D32, D34 to D33, D35 to D34, D36 to D35, D37 to D36, D38 to D37, D39 to D38, D40 to D39, D41 to D40, D42 to D41, D43 to D42, D44 to D43, D45 to D44, D46 to D45, D47 to D46, D48 to D47, D49 to D48, D13 to RD1
Connections:
- net 3v3: now also C1.1, R1.1, R2.1
- net col2: no longer D1.1 (K), D10.1 (K), D11.1 (K), D12.1 (K), D2.1 (K), D3.1 (K), D4.1 (K), D5.1 (K), D6.1 (K), D7.1 (K), D8.1 (K), D9.1 (K), RD1.1 (K), U1.1 (PA02_A0_D0)
- net gnd: now also C1.2
- net scl: now also R1.2
- net sda: now also R2.2
- new net row0: D1.1 (K), D10.1 (K), D11.1 (K), D12.1 (K), D2.1 (K), D3.1 (K), D4.1 (K), D5.1 (K), D6.1 (K), D7.1 (K), D8.1 (K), D9.1 (K), RD1.1 (K), U1.1 (PA02_A0_D0)
- no-connect marks 10 -> 11
Other:
- note added: "Decoupling Capacitor (trys to prevent brownouts)"
- note added: "I2C Pullup Resistors (required if no OLED)"
- moved on the sheet: SW42, SW49, SW50, SW51, U3
